File: pcb/snowhackpad.kicad_pcb (KiCad board)
At the start: 2 copper layers, 119.9 x 85.6 mm, 10 parts, among them J1 Conn_01x04, SW1 SW_Push, SW2 SW_Push, SW3 SW_Push, SW4 SW_Push, SW5 RotaryEncoder_Switch, U1 XIAO-RP2040-DIP

Commit message: Update: Update Kicad PCB
Parts:
- added G***: LOGO, LOGO, F.Cu at (131.9, 131.0)
- added G***: LOGO, LOGO, F.Cu at (227.5, 129.4)
Other:
- board text added: "coolest hackpad by alex (TM)"
- board text removed: "Alex's Hackpad V1"
- board text removed: "Blueprint by Hack Club"
